Commit message: Add files via upload

File: description/lidar.xacro (robot description, xacro)
@@ -4,5 +4,5 @@
         <parent link="chassis"/>
         <child link="laser_frame"/>
-        <origin xyz="0.375 0 0.76" rpy="0 0 0"/>
+        <origin xyz="0.375 0 0.775" rpy="0 0 0"/>
     </joint>
     <link name="laser_frame">

File: description/robot.urdf.xacro (robot description, xacro)
@@ -2,6 +2,6 @@
 <robot xmlns:xacro="http://www.ros.org/wiki/xacro"  name="robot">
     <xacro:include filename="robot_core.xacro" />
-    <!-- <xacro:include filename="gazebo_control.xacro" /> -->
-    <xacro:include filename="ros2_control.xacro" />
+    <xacro:include filename="gazebo_control.xacro" />
+    <!-- <xacro:include filename="ros2_control.xacro" /> -->
     <xacro:include filename="lidar.xacro" />
     <xacro:include filename="camera.xacro" />

File: description/robot_core.xacro (robot description, xacro)
@@ -35,5 +35,5 @@
     </link>
     <!-- BASE_FOOTPRINT LINK -->
-    <!-- <joint name="base_footprint_joint" type="fixed">
+    <joint name="base_footprint_joint" type="fixed">
         <parent link="base_link"/>
         <child link="base_footprint"/>
@@ -41,5 +41,5 @@
     </joint>
     <link name="base_footprint">
-    </link> -->
+    </link>
     <!-- CHASSIS LINK -->
     <joint name="chassis_joint" type="fixed">
